Commit message: robot nav sim

File: description/lidar.xacro (robot description, xacro)
@@ -1,4 +1,4 @@
 <?xml version="1.0"?>
-<robot xmlns:xacro="http://www.ros.org/wiki/xacro">
+<robot xmlns:xacro="http://www.ros.org/wiki/xacro" >
     <joint name="laser_joint" type="fixed">
         <parent link="chassis"/>
@@ -12,10 +12,4 @@
             </geometry>
             <material name="black"/>
-        </visual>
-        <visual>
-            <origin xyz="0 0 -0.04"/>
-            <geometry>
-                <box size="0.1 0.1 0.05"/>
-            </geometry>
         </visual>
         <collision>
@@ -31,5 +25,5 @@
         <material>Gazebo/Black</material>
         <sensor name="laser" type="ray">
-            <pose>0 0 0 0 0 0</pose>
+            <pose> 0 0 0 0 0 0 </pose>
             <visualize>false</visualize>
             <update_rate>10</update_rate>
@@ -47,5 +41,5 @@
                 </range>
             </ray>
-            <plugin name="laser_controller" filename="libgasebo_ros_ray_sensor.so">
+            <plugin name="laser_controller" filename="libgazebo_ros_ray_sensor.so">
                 <ros>
                     <argument>~/out:=scan</argument>
